File: hardware/sn64/cart-interface.kicad_sch (KiCad schematic)
At the start: 72 parts, among them Q201 2N7002, U201 SN74LVC4245APWR, U202 SN74LVC4245APWR, U203 SN74LVC4245APWR, U204 SN74LVC4245APWR, U205 SN74LVC4245APWR, U206 SN74LVC4245APWR, U207 SN74LVC4245APWR, U209 SN74LVC244APWR, U210 SN74LVC1G07DBVR, U211 SN74LVC1G07DBVR, U212 SN74LVC1G07DBVR, U213 SN74LVC1G06DBVR, U214 SN74LVC1G06DBVR

Commit message: Board top with real ECP5 clocks; header region probe, flash boot ROM, CIC pin fix
- sn64_board_top: EHXPLLL 25->62.5 MHz and pixel x5, one glitchless DCSC
  (NEG mode) that selects NTSC/PAL and starts/stops the SNES clock, bootstrap
  ROM from the configuration flash via USRMCLK, CIC pad DIR sequencing.
  Routed on the 85F with trial pins: all five clocks pass, 143/208 BRAM.
- ROM-header region fallback (sn64_header_probe + socket mux) merged into
  sn64_top; priority forced > key CIC > valid header > NTSC. tb_system now
  also runs with an EU header and must start in PAL.
- Bootstrap ROM window from SPI flash (SummerCart64 memory_flash, unmodified).
- Cart sheet rev 0.3.1: per-pin SN74LVC1T45 for CIC data; sn64_cic_pad and
  tb_cic_pad with a fault build.
- Bridge data octet enable/direction gated by permit combinationally.
- evaluate.py --mode sim: all 30 results pass, including fault injections.

Co-Authored-By: Claude Fable 5.1 <noreply@anthropic.com>
Parts:
- added C230, C231: 100nF, Capacitor_SMD:C_0603_1608Metric, symbol Device:C
- added C232, C233: 10uF 10V, Capacitor_SMD:C_0805_2012Metric, symbol Device:C
- added R215: 33, Resistor_SMD:R_0603_1608Metric, symbol Device:R
- added R216, R217, R220, R221: 10k, Resistor_SMD:R_0603_1608Metric, symbol Device:R
- added R218, R219: 100k, Resistor_SMD:R_0603_1608Metric, symbol Device:R
- added U215, U216: SN74LVC1T45DBVR, Package_TO_SOT_SMD:SOT-23-6, symbol Logic_LevelTranslator:SN74LVC1T45DBV
- C228, C229: value 10uF 10V -> 100nF; footprint Capacitor_SMD:C_0805_2012Metric -> Capacitor_SMD:C_0603_1608Metric
- R214: value 100k -> 33
Connections:
- net cic_data0_out is gone; now on net GND: U206.18 (B4)
- net GND: now also U209.11 (2A1), U209.8 (1A4), C230.2, C231.2, C232.2, C233.2, R216.2, R217.2, R218.2, R219.2, R220.2, R221.2, U215.2 (GND), U216.2 (GND); no longer R214.2
- net INTERFACE_3V3: now also C228.1, C230.1, C233.1, U215.1 (VCCA), U216.1 (VCCA); no longer C229.1
- net SNES_5V_CART: now also C229.1, C231.1, C232.1, U215.6 (VCCB), U216.6 (VCCB); no longer C228.1
- net SNES_CIC_DATA0: now also R214.2, R216.1; no longer RN211.5 (R4.2), U209.11 (2A1)
- net SNES_CIC_DATA1: now also R215.2, R217.1; no longer R214.1, U209.8 (1A4)
- net XA_CIC_DATA0: no longer names the net of U206.6 (A4)
- net XA_CIC_DATA0: no longer RN211.4 (R4.1)
- net cic_data0_sense: no longer names the net of U209.9 (2Y1)
- net cic_data1_in: no longer names the net of U209.12 (1Y4)
- new net XB_CIC_DATA0: R214.1, U215.4 (B)
- new net XB_CIC_DATA1: R215.1, U216.4 (B)
- new net cic_data0: R218.1, U215.3 (A)
- new net cic_data0_dir: R220.1, U215.5 (DIR)
- new net cic_data1: R219.1, U216.3 (A)
- new net cic_data1_dir: R221.1, U216.5 (DIR)
- no-connect marks 10 -> 15
Other:
- note added: "CIC DATA PINS - PER-PIN DIRECTION CONTROL (J2.55 CIC_DATA0 via U215, J2.24 CIC_DATA1 via U216)"
- note added: "DRAFT 0.3.1-cart: schematic circuit candidate only. No PCB, SI simulation, power sequencing test, ESD part or cartridge test has been performed. SNES_5V_CART and INTERFACE_3V3 are hierarchical inputs from the (future) power sheet; #FLG201/#FLG202 mark them externally supplied for ERC only. Open: socket ESD array selection, final damping/pull values (CIC pull-down value to confirm against a real k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"
- note added: "PULL/BIAS: /IRQ, /RESET, EXPAND 10k to cartridge 5 V (OpenSFC keeps pull-ups on IRQ/EXPAND); CIC_DATA0/1 10k pull-downs (R216/R217). Values provisional."
- note added: "SN74LVC1T45 (TI SCES515N): A = FPGA side (VCCA = INTERFACE_3V3), B = cartridge side (VCCB = SNES_5V_CART). No shared enable. DIR is referenced to VCCA and driven directly by its own FPGA pin cic_dataN_dir: H = A->B (FPGA drives the cartridge), L = B->A (listen). FPGA rule (no OE pin, SCES515N 8.2.2): set DIR high BEFORE driving cic_dataN; switch cic_dataN to input BEFORE setting DIR low. Idle: R2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"
- note added: "U201-U206: console outputs, DIR strapped to GND (fixed FPGA->cartridge). U201-U205 share CTL_OE_N_5V (bridge ctl_oe_n); U206 (SYSTEM_CLK + CIC_CLK + CIC_SLAVE_RESET only) has its own CIC_OE_N_5V (sn64_top snes_cic_oe_n, enabled from the sequencer IFACE state). U207: D0-D7, DIR and OE both FPGA-controlled (bridge data_dir / data_oe_n). Unused B inputs tied to GND; unused A outputs no-connect."
- note added: "U209 SN74LVC244A at 3.3 V: 5.5 V-tolerant inputs with Ioff; receives /IRQ, /RESET, EXPAND (CIC data pins use U215/U216). U210-U212 74LVC1G07 / U213 74LVC1G06: 3.3 V open-drain outputs (5.5 V tolerant, Ioff) pulled to SNES_5V_CART. No 5 V pull-up reaches an FPGA pin. Interface rail off or FPGA unconfigured => every translator /OE released high (isolated). /RESET: Q201 open-drain sink. RESET_GATE_5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"
- note removed: "DRAFT 0.3-cart: schematic circuit candidate only. No PCB, SI simulation, power sequencing test, ESD part or cartridge test has been performed. SNES_5V_CART and INTERFACE_3V3 are hierarchical inputs from the (future) power sheet; #FLG201/#FLG202 mark them externally supplied for ERC only. Open: socket ESD array selection, independent CIC_DATA0 release, SuperCIC pair-mode drive on CIC_DATA1, final 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"
- note removed: "PULL/BIAS: /IRQ, /RESET, EXPAND 10k to cartridge 5 V (OpenSFC keeps pull-ups on IRQ/EXPAND); CIC_DATA1 100k idle bias. Values provisional."
- note removed: "U201-U206: console outputs, DIR strapped to GND (fixed FPGA->cartridge). U201-U205 share CTL_OE_N_5V (bridge ctl_oe_n); U206 (SYSTEM_CLK + CIC_CLK/SLAVE_RESET/DATA0) has its own CIC_OE_N_5V (proposed bridge port cic_oe_n). U207: D0-D7, DIR and OE both FPGA-controlled (bridge data_dir / data_oe_n). Unused B inputs tied to GND; unused A outputs no-connect."
- note removed: "U209 SN74LVC244A at 3.3 V: 5.5 V-tolerant inputs with Ioff; receives /IRQ, /RESET, EXPAND, CIC_DATA1 and CIC_DATA0 (sense while released). U210-U212 74LVC1G07 / U213 74LVC1G06: 3.3 V open-drain outputs (5.5 V tolerant, Ioff) pulled to SNES_5V_CART. No 5 V pull-up reaches an FPGA pin. Interface rail off or FPGA unconfigured => every translator /OE released high (isolated). /RESET: Q201 open-drain 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"
- moved on the sheet: C216, C217, C218, C219, C220, C221, C222, C223, C224, C225, C226, C227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
