File: hardware/sn64/sn64.kicad_sch (KiCad schematic)
At the start: 2 parts, among them J1 N64_Cartridge_Edge_50, J2 SNES_Female_Slot_62

Commit message: Board top with real ECP5 clocks; header region probe, flash boot ROM, CIC pin fix
- sn64_board_top: EHXPLLL 25->62.5 MHz and pixel x5, one glitchless DCSC
  (NEG mode) that selects NTSC/PAL and starts/stops the SNES clock, bootstrap
  ROM from the configuration flash via USRMCLK, CIC pad DIR sequencing.
  Routed on the 85F with trial pins: all five clocks pass, 143/208 BRAM.
- ROM-header region fallback (sn64_header_probe + socket mux) merged into
  sn64_top; priority forced > key CIC > valid header > NTSC. tb_system now
  also runs with an EU header and must start in PAL.
- Bootstrap ROM window from SPI flash (SummerCart64 memory_flash, unmodified).
- Cart sheet rev 0.3.1: per-pin SN74LVC1T45 for CIC data; sn64_cic_pad and
  tb_cic_pad with a fault build.
- Bridge data octet enable/direction gated by permit combinationally.
- evaluate.py --mode sim: all 30 results pass, including fault injections.

Co-Authored-By: Claude Fable 5.1 <noreply@anthropic.com>
Connections:
- no-connect marks 26 -> 27
Other:
- sheet SNES cartridge interface ports: added cic_data0, cic_data0_dir, cic_data1, cic_data1_dir; removed cic_data0_out, cic_data0_sense, cic_data1_in
