File: hardware/sn64/usb-programmer.kicad_sch (KiCad schematic)
At the start: 41 parts, among them J101 DX07S016JA3R1500, J102 JTAG_SERVICE, U101 USBLC6-2SC6, U102 USBLC6-2SC6, U103 AP2112K-3.3TRG1, U104 FT232HL (rev C), U105 SN74AXC4T774PWR, U106 93AA56BT-I/OT (DNP), Y101 ABM3B-12.000MHZ-10-1-U-T

Commit message: Complete schematic draft: FPGA, power, clock/HDMI/audio sheets; PAL HDMI; cart audio
- New child sheets attached and wired at the root: FPGA (all 381 balls,
  W25Q128JV config flash, JTAG to the USB programmer, N64 edge through
  host-gated bus switches), power (priority-muxed host/USB eFuses, TUSB320
  permission, TPS63070 5V_PRE, FPGA bucks, cartridge eFuse and monitors),
  clock/HDMI/audio (Si5351A, TPD12S016 HDMI, PCM1808 cartridge-audio ADC).
- Real pinout: fpga/constraints/sn64_board.lpf; board top routed with it,
  all five clocks pass (SNES 28.9 MHz vs 21.48 required).
- PAL HDMI 576p50 frame-locked to the PAL SNES; Si5351 CLK2 retargeted only
  while the SNES clock is stopped. Cartridge audio mixed into HDMI.
  REGION_INFO/REGION_SOURCE mailbox telemetry shown in the menu.
  tb_system runs NTSC default, PAL header, PAL key and NTSC key.
- Safety fixes: efuse_fault_n pulled up to FPGA_3V3 (a 5V_PRE divider would
  back-drive a non-hot-socket bank); cart enable pull-ups 10k -> 4.7k
  (ECP5 config-time pull-down up to 150 uA).
- Checks: ERC 0 errors; interfaces 30/30, USB 69/69, cart 20/20, FPGA 13/13,
  power 23/23, A/V 30/30, root connectivity 4/4, all negative tests caught;
  evaluate.py --mode sim passes.

Co-Authored-By: Claude Fable 5.1 <noreply@anthropic.com>
Parts:
- R101, R102: now not fitted
Connections:
- net JTAG_TCK renamed jtag_tck
- net JTAG_TDI renamed jtag_tdi
- net JTAG_TDO renamed jtag_tdo
- net JTAG_TMS renamed jtag_tms
Other:
- note added: "TARGET_VREF comes from FPGA_3V3 (VCCIO8) through R414 on the FPGA sheet. It powers the B-side translator; it is NOT a USB power output. jtag_tck/tms/tdi/tdo go to the ECP5 dedicated JTAG balls (FPGA sheet). Only one programmer may own JTAG at a time."
- note added: "USB_3V3 powers this programmer and the power sheet TUSB320 (U301) only. No USB/host power tie. USB_VBUS also feeds the power sheet default-off USB input (U302); R101/R102 DNP, U301 presents Rd. USB suspend, inrush, ESD and power-off behavior require bench tests."
- note removed: "TARGET_VREF comes from the future FPGA programming rail. It powers the B-side translator; it is NOT a USB power output. JTAG_TCK/TDI/TDO/TMS need final FPGA/flash integration. Only one programmer may own JTAG at a time."
- note removed: "USB_3V3 powers this programmer only. No USB/host power tie. Main FPGA/system power and cartridge power remain separate work. USB suspend, inrush, ESD and power-off behavior require bench tests."
