File: hardware/sn64/av-clock.kicad_sch (KiCad schematic)
At the start: 50 parts, among them J701 HDMI_A 10029449-111RLF, U701 Si5351A-B-GTR, U702 TPD12S016PWR, U703 PCM1808PWR, X701 25MHz CJO05-250003320B30, X702 12.288MHz CJO05-122883320B30, Y701 25MHz 10pF

Commit message: Remove the on-board HDMI output: the console's own output is the only video path
Owner decision 2026-09-29: the SNES picture and sound reach the TV through the
console (M64 HDMI, N64 AV jack) via the cartridge-bus frame window; the board
has no video output of its own.

FPGA: delete sn64_av_out/av_hdmi_tx/av_serializer, tb_av_out and the vendored
hdl-util/hdmi tree; sn64_clock_init keeps CLK2 powered down (reg 3 = 0xFC) and
writes nothing after start-up; board top keeps one PLL, drops si_clk2/hdmi_*.
Sim suite 38/38; routed 203/208 DP16KD, 113 I/O, 41 % logic, all clocks pass.

Schematic: FPGA sheet rev 0.5-fpga (TMDS/HPD/DDC/si_clk2 pins removed, LPF and
CSV regenerated), A/V sheet draft 0.2-av (J701, TPD12S016, TMDS coupling, R705
gone; Si5351 pin 6 open), root sheet symbols re-packed. ERC 0 errors; all
sheet checks and negative tests pass (FPGA 14/14, A/V 27/27 with new checks).

Board: rebuilt from the new netlist (410 parts, 530 nets), FPGA-support zone
widened; DRC clean apart from the by-design USB-C edge pads and the N64 finger
mask opening. Power budget rows for the HDMI loads removed. Docs updated;
av-output-implementation.md is now the retirement record.

Co-Authored-By: Claude Fable 5.1 <noreply@anthropic.com>
Parts:
- removed C704, C705, C706, C707, C708, C709, C710, C711: 22nF, Capacitor_SMD:C_0603_1608Metric, symbol Device:C
- removed C712, C713, C714: 100nF, Capacitor_SMD:C_0603_1608Metric, symbol Device:C
- removed J701: HDMI_A 10029449-111RLF, Connector_Video:HDMI_A_Amphenol_10029449-x01xLF_Horizontal, symbol Connector:HDMI_A
- removed R705: 0R, Resistor_SMD:R_0603_1608Metric, symbol Device:R
- removed TP701: CEC_A, TestPoint:TestPoint_Pad_D1.0mm, symbol Connector:TestPoint
- removed U702: TPD12S016PWR, Package_SO:TSSOP-24_4.4x7.8mm_P0.65mm, symbol SN64_AV:TPD12S016PW
Connections:
- net SI_CLK2_SRC: no longer names the net of U701.6 (CLK2)
Other:
- note added: "CLOCKS (docs/design/clock-plan.md). U701 Si5351A-B-GT (Skyworks Si5351-B Rev 1.3): CLK0 = NTSC master 21.4772727 MHz, CLK1 = PAL master 21.28137 MHz; CLK2 powered down and disabled (register 3 = 0xFC), pin 6 open; programmed at power-on by fpga/rtl/sn64_clock_init.sv over si_scl/si_sda (I2C address 0x60, 400 kHz). VDD and VDDO both FPGA_3V3 (sec. 7.2: VDDO with or before VDD). One 100 nF per supp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"
- note added: "DRAFT 0.2-av: schematic circuit candidate only. No PCB, SI simulation or audio measurement has been performed. FPGA_3V3 and 5V_PRE are hierarchical inputs from the power sheet (ERC origins there: #FLG304 and the TPS63070 VOUT). Provisional: 0R series values, 200 R console-equivalent load (OpenSFC value, verify on SHVC-CPU-01), X7R 1 uF coupling, footprints of X701/X702. Sources and SHA-256 of eve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"
- note added: "SN 64 - CLOCKS AND CARTRIDGE AUDIO ADC (DRAFT 0.2-av)"
- note added: "VIDEO AND AUDIO TO THE CONSOLE (docs/design/console-video-path.md): the SNES picture and sound reach the N64/M64 over the cartridge bus (N64 endpoint frame window) and are shown on the console's own output (N64 AV jack, M64 HDMI). This board has no video output of its own. The HDMI section of draft 0.1-av (J701 type-A, U702 TPD12S016, 22 nF TMDS coupling, Si5351 CLK2 pixel clock) was removed in 0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"
- note removed: "CLOCKS (docs/design/clock-plan.md). U701 Si5351A-B-GT (Skyworks Si5351-B Rev 1.3): CLK0 = NTSC master 21.4772727 MHz, CLK1 = PAL master 21.28137 MHz, CLK2 = HDMI pixel 27.0197947 MHz; programmed at power-on by fpga/rtl/sn64_clock_init.sv over si_scl/si_sda (I2C address 0x60, 400 kHz). VDD and VDDO both FPGA_3V3 (sec. 7.2: VDDO with or before VDD). One 100 nF per supply pin (sec. 7.1). Y701 25 MHz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"
- note removed: "DRAFT 0.1-av: schematic circuit candidate only. No PCB, SI simulation, HDMI compliance or audio measurement has been performed. FPGA_3V3 and 5V_PRE are hierarchical inputs from the power sheet (ERC origins there: #FLG304 and the TPS63070 VOUT). Provisional: 0R series values, 200 R console-equivalent load (OpenSFC value, verify on SHVC-CPU-01), X7R 1 uF coupling, footprints of J701/X701/X702. Sour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"
- note removed: "HDMI (docs/design/av-output-implementation.md): 720x480p, ECP5 LVCMOS33D pseudo-differential outputs. TMDS network reused from ULX3S gpdi.sch @6a92cec (MIT + logo condition, hardware/sn64/THIRD_PARTY.md): each TMDS line = 22 nF series capacitor (ULX3S C38-C45), no series resistor. U702 TPD12S016 (TI SLLSE96F) on the connector side: TMDS ESD, DDC/CEC level shift (A = FPGA_3V3, B = 5V_OUT), HPD buf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"
- note removed: "SN 64 - CLOCKS, HDMI OUTPUT AND CARTRIDGE AUDIO ADC (DRAFT 0.1-av)"
- title: SN 64 - clocks, HDMI and cartridge audio -> SN 64 - clocks and cartridge audio
