File: hardware/sn64/fpga.kicad_sch (KiCad schematic)
At the start: 95 parts, among them U401 LFE5U-85F-6BG381C, U402 SN74CB3Q3384APWR, U403 SN74CB3Q3384APWR, U404 SN74CB3Q3384APWR, U405 W25Q128JVSIQ, U406 SN74LVC1G14DBVR, U407 SN74LVC1G07DBVR

Commit message: Remove the on-board HDMI output: the console's own output is the only video path
Owner decision 2026-09-29: the SNES picture and sound reach the TV through the
console (M64 HDMI, N64 AV jack) via the cartridge-bus frame window; the board
has no video output of its own.

FPGA: delete sn64_av_out/av_hdmi_tx/av_serializer, tb_av_out and the vendored
hdl-util/hdmi tree; sn64_clock_init keeps CLK2 powered down (reg 3 = 0xFC) and
writes nothing after start-up; board top keeps one PLL, drops si_clk2/hdmi_*.
Sim suite 38/38; routed 203/208 DP16KD, 113 I/O, 41 % logic, all clocks pass.

Schematic: FPGA sheet rev 0.5-fpga (TMDS/HPD/DDC/si_clk2 pins removed, LPF and
CSV regenerated), A/V sheet draft 0.2-av (J701, TPD12S016, TMDS coupling, R705
gone; Si5351 pin 6 open), root sheet symbols re-packed. ERC 0 errors; all
sheet checks and negative tests pass (FPGA 14/14, A/V 27/27 with new checks).

Board: rebuilt from the new netlist (410 parts, 530 nets), FPGA-support zone
widened; DRC clean apart from the by-design USB-C edge pads and the N64 finger
mask opening. Power budget rows for the HDMI loads removed. Docs updated;
av-output-implementation.md is now the retirement record.

Co-Authored-By: Claude Fable 5.1 <noreply@anthropic.com>
Connections:
- net hdmi_ck_n: no longer names the net of U401.B18 (PT116B)
- net hdmi_ck_p: no longer names the net of U401.A17 (PT116A)
- net hdmi_d0_n: no longer names the net of U401.B16 (PT110B)
- net hdmi_d0_p: no longer names the net of U401.A16 (PT110A)
- net hdmi_d1_n: no longer names the net of U401.C14 (PT83B)
- net hdmi_d1_p: no longer names the net of U401.A14 (PT83A)
- net hdmi_d2_n: no longer names the net of U401.A13 (PT76B)
- net hdmi_d2_p: no longer names the net of U401.A12 (PT76A)
- net hdmi_hpd: no longer names the net of U401.E13 (PT80B)
- net hdmi_scl: no longer names the net of U401.D15 (PT107A)
- net hdmi_sda: no longer names the net of U401.E15 (PT107B)
- net si_clk2: no longer names the net of U401.F2 (PL44C)
- no-connect marks 98 -> 110
Other:
- note added: "DRAFT 0.5-fpga: schematic only - no PCB, no SI or power-integrity analysis, no hardware test. FPGA_1V1/2V5/3V3 come from the power sheet (its #FLG302-#FLG304 are their ERC origins). #FLG404 marks FPGA_VCCAUX, fed only through FB401. Pin map: interfaces/fpga-pin-map.csv; constraints: fpga/constraints/sn64_board.lpf; doc: docs/design/fpga-schematic.md."
- note added: "Rails: VCC = FPGA_1V1 (1.1 V, DS-02012 Table 3.2), VCCAUX = FPGA_2V5 through FB401 (TN-02038 Figure 3.1), every VCCIO0/1/2/3/6/7/8 = FPGA_3V3. Bank plan: 0 = N64 PI/CIC/SI behind the bus switches (top bank, hot-socket capable), 1 = spare (HDMI removed in 0.5-fpga: video goes to the console over the cartridge bus), 2+3 = cartridge translators B side, 6+7 = clocks, Si5351 I2C, ADC, power control, L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"
- note removed: "DRAFT 0.4-fpga: schematic only - no PCB, no SI or power-integrity analysis, no hardware test. FPGA_1V1/2V5/3V3 come from the power sheet (its #FLG302-#FLG304 are their ERC origins). #FLG404 marks FPGA_VCCAUX, fed only through FB401. Pin map: interfaces/fpga-pin-map.csv; constraints: fpga/constraints/sn64_board.lpf; doc: docs/design/fpga-schematic.md."
- note removed: "Rails: VCC = FPGA_1V1 (1.1 V, DS-02012 Table 3.2), VCCAUX = FPGA_2V5 through FB401 (TN-02038 Figure 3.1), every VCCIO0/1/2/3/6/7/8 = FPGA_3V3. Bank plan: 0 = N64 PI/CIC/SI behind the bus switches (top bank, hot-socket capable), 1 = HDMI LVCMOS33D + DDC/HPD, 2+3 = cartridge translators B side, 6+7 = clocks, Si5351 I2C, ADC, power control, LED, 8 = configuration flash. GND: all 113 GND balls (the L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"
