File: hardware/sn64-v2/fpga.kicad_sch (KiCad schematic)
At the start: 92 parts, among them U1 LFE5U-85F-8BG381I, U2 W25Q128JVSIQ, U3 TPS3808G01DBVR, U6 TLA2528IRTER, X1 27MHz 1631-27005-BTBEYA

Commit message: A game through the board's own wiring; two wiring rules corrected from the data sheets
The owner's game now runs through a model of the v2 board that is generated
from the board file: the real top level on its balls, a model of every part on
its pads with the makers' pin numbers, the cartridge on the socket's pins and
the N64 on the edge fingers (make_board_sim.py, tb_board_game.sv,
run_game.py --board).

Found by reading each maker's data sheet, corrected on the board:
- U204's socket-to-FPGA byte was enabled all the time, also while its 5 V side
  has no supply. It now has an enable of its own (SENSE_OE_N, R214).
- The supply converter's address pin was tied to ground; the sheet gives the
  address the logic uses for the pin left open.

Found by the board run, corrected in the logic:
- the status LED was dark in a game;
- the cartridge's pins were loose for a moment at start and at power-off. They
  are now held at rest while the cartridge has its 5 V, and /RESET is held 1 ms
  before the 5 V goes.

Wiring check 21 of 21, 20 of 20 deliberate mistakes caught. The board run
refuses a reversed cartridge and two deliberately mis-wired boards. The logic
suite passes with two new fault builds; the design routes with every clock
passing. Test set results: 38 of 38 judged programs pass.

Still open before an order: six unrouted connections, the socket sample, the
first load of a blank board (docs/design/board-verification.md).

Co-Authored-By: Claude Opus 5.5 <noreply@anthropic.com>
Parts:
- U6: Note ADDR=GND; AIN4 = FPGA_1V1 direct; footprint EP size to veri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 -> ADDR open: I2C address 0x10 (SBAS961A table 2: no resistor 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
Connections:
- net GND: no longer U6.11 (ADDR)
- net L_EXPAND renamed SENSE_OE_N
- no-connect marks 105 -> 106
Changed lines of the file:
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@@
 (no_connect (at 370.84 147.32))
 (wire (pts (xy 370.84 142.24) (xy 365.76 142.24)) (stroke (width 0) (type default)))
-(global_label "L_EXPAND" (shape passive) (at 365.76 142.24 180) (fields_autoplaced yes) (effects (font (size 1.016 1.016)) (justify right)) (property "Intersheetrefs" "${INTERSHEET_REFS}" (at 365.76 142.24 0) (effects (font (size 1.27 1.27)) (hide yes))))
+(global_label "SENSE_OE_N" (shape passive) (at 365.76 142.24 180) (fields_autoplaced yes) (effects (font (size 1.016 1.016)) (justify right)) (property "Intersheetrefs" "${INTERSHEET_REFS}" (at 365.76 142.24 0) (effects (font (size 1.27 1.27)) (hide yes))))
 (wire (pts (xy 370.84 134.62) (xy 365.76 134.62)) (stroke (width 0) (type default)))
 (global_label "L_PA2" (shape passive) (at 365.76 134.62 180) (fields_autoplaced yes) (effects (font (size 1.016 1.016)) (justify right)) (property "Intersheetrefs" "${INTERSHEET_REFS}" (at 365.76 134.62 0) (effects (font (size 1.27 1.27)) (hide yes))))
@@
 (property "LCSC" "C2866175" (at 67.31 441.96 0) (effects (font (size 1.27 1.27)) (hide yes)))
 (property "MPN" "TLA2528IRTER" (at 67.31 441.96 0) (effects (font (size 1.27 1.27)) (hide yes)))
-(property "Note" "ADDR=GND; AIN4 = FPGA_1V1 direct; footprint EP size to verify against SBAS961A mechanical drawing" (at 67.31 441.96 0) (effects (font (size 1.27 1.27)) (hide yes)))
+(property "Note" "ADDR open: I2C address 0x10 (SBAS961A table 2: no resistor on ADDR; straight to ground is not a listed setting); AIN4 = FPGA_1V1 direct; footprint EP size to verify against SBAS961A mechanical drawing" (at 67.31 441.96 0) (effects (font (size 1.27 1.27)) (hide yes)))
 (pin "15")
 (pin "16")
@@
 (wire (pts (xy 85.09 435.61) (xy 90.17 435.61)) (stroke (width 0) (type default)))
 (global_label "ADC_SDA" (shape passive) (at 90.17 435.61 0) (fields_autoplaced yes) (effects (font (size 1.016 1.016)) (justify left)) (property "Intersheetrefs" "${INTERSHEET_REFS}" (at 90.17 435.61 0) (effects (font (size 1.27 1.27)) (hide yes))))
-(wire (pts (xy 85.09 438.15) (xy 90.17 438.15)) (stroke (width 0) (type default)))
-(global_label "GND" (shape passive) (at 90.17 438.15 0) (fields_autoplaced yes) (effects (font (size 1.016 1.016)) (justify left)) (property "Intersheetrefs" "${INTERSHEET_REFS}" (at 90.17 438.15 0) (effects (font (size 1.27 1.27)) (hide yes))))
+(no_connect (at 85.09 438.15))
 (wire (pts (xy 85.09 440.69) (xy 90.17 440.69)) (stroke (width 0) (type default)))
 (global_label "ADC_DECAP" (shape passive) (at 90.17 440.69 0) (fields_autoplaced yes) (effects (font (size 1.016 1.016)) (justify left)) (property "Intersheetrefs" "${INTERSHEET_REFS}" (at 90.17 440.69 0) (effects (font (size 1.27 1.27)) (hide yes))))

Commit message: USB loader chip (FT231X on JTAG), USB-C on the player's right, no USB logic in the FPGA; board copper complete
The owner: "Add back just the usb loader chip and put the usb on the right side of the cart",
and of the FPGA's own USB logic: "no i want it clean so remove it".

Board (hardware/sn64-v2)
- U13 FT231XS between the USB-C socket and the FPGA's JTAG port, wired like the ULX3S so that
  openFPGALoader drives it as it is (-b ulx3s): TCK on DSR#, TMS on DCD#, TDI on RI#, TDO on CTS#.
  Bus-powered as FTDI's data sheet draws it; with no cable it has no supply.
- Six small parts with it: three 100 nF, two 47 pF, and the 4.7 k pull-down on TCK that Lattice
  asks for. R19 and R20 are its 27 ohm series resistors now; R21 and R201 are gone. 182 parts.
- The socket, its protection part and the VBUS capacitor are on the -X edge, the player's right.
- apply_usb_loader_v2.py carries it into the routed board: 19 nets routed with everything else
  locked, a keep-out under the socket's body. VBUS to the input switch: 55 mm, was 104 mm.
- close_open_items_v2.py closes what KiCad's check still listed: the N64 controller line (a
  leftover via), the converter's 3.3 V pin, flash D2 at the corner of the ball grid (laid again
  together with its two neighbours) and five ground pads with a single thermal spoke (now solid).
  KiCad's rule check: no error, no open connection, 217 of 217 signal nets.
- Wiring check: 22 of 22; 25 of 25 deliberate mistakes caught, five of them new.

FPGA (fpga/)
- The USB device, its two clocks, its share of the flash and the reboot line are out of the
  logic, with the TinyFPGA core and the two tools that prepared it. The flash reader is
  SummerCart64's memory_flash unmodified again. 28,955 LUT4 (30,820 before), 107 pins (111),
  4 clocks (6).
- evaluate.py --mode sim passes; every clock passes on the board's pins.
- The game run of 660 pictures is the same as before, picture for picture, and the sound byte
  for byte.

Board-level runs on the new boa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
Parts:
- removed R19, R20: 22, Resistor_SMD:R_0603_1608Metric, symbol Device:R
- removed R21: 1.5k, Resistor_SMD:R_0603_1608Metric, symbol Device:R
- added R41: 4.7k, Resistor_SMD:R_0603_1608Metric, symbol Device:R
Connections:
- net GND: now also R41.1
- net JTAG_TCK: now also R41.2
- net PROGRAMN_PULL: no longer names the net of U1.C9 (PT54A)
- net USB_DN_F: no longer names the net of U1.C13 (PT78B)
- net USB_DP_F: no longer names the net of U1.C12 (PT71B)
- net USB_PU: no longer names the net of U1.C14 (PT83B)
- no-connect marks 106 -> 110
Other:
- note added: "SN64 v2 FPGA SHEET - LFE5U-85F CABGA381 (-8BG381I, Mouser stock), configuration flash, 27 MHz clock, JTAG, telemetry ADC, reset supervisor. Pin map: interfaces/fpga-pin-map.csv (tools/pin_plan.py): every signal on rings 1-3; constraints fpga/constraints/sn64_board.lpf."
- note removed: "SN64 v2 FPGA SHEET - LFE5U-85F CABGA381 (-8BG381I, Mouser stock), configuration flash, 27 MHz clock, USB device pins, telemetry ADC, reset supervisor. Pin map: interfaces/fpga-pin-map.csv (tools/pin_plan.py): every signal on rings 1-3; constraints fpga/constraints/sn64_board.lpf."
- moved on the sheet: C34, C35, C36, C37, C38, C39, C40, R22, R23, R24, R25, R26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

Commit message: Pre-order review, work in progress: finger fill, U6 footprint, USB-C port from the drawings, parts list numbers, power re-layout started
Checkpoint in the middle of the review, committed at the owner's request. Not a release.

Done and on the board file:
- ground fill taken out of the N64 edge fingers, ground plane extended to the finger vias
  (apply_finger_clearance_v2.py)
- U6 footprint with the exposed pad of its data sheet, R17 moved, leftovers of the first
  routing trimmed, silkscreen labels tidied, part records synced with the schematic
- USB supply capacitance 8.0 uF, selector soft-start 10 nF

Done elsewhere:
- shell: USB-C port from the JAE drawing, the USB-IF plug limits and the SummerCart64 port
- a maker part number on every bought part; yellow-green lamp; 1 uF at each ADC supply pin
- pack_bitstream.py: the FPGA image packed for a fast load, and the whole flash as one file
- make_production_v2.py (its output is not in this commit: it is remade when the board is done)

In progress, schematic ahead of the board:
- the schematic has 12 more small parts (R321, C324, C325, C213-C220, C46) that the makers'
  data sheets ask for; the board file does not have them yet
- apply_power_layout_v2.py and make_power_plan.py lay the power section out again by the
  makers' layout rules; so far only on working copies under build/

Co-Authored-By: Claude Opus 5.5 <noreply@anthropic.com>
Parts:
- added C46: 1uF, Capacitor_SMD:C_0603_1608Metric, symbol Device:C
- C1, C11, C12, C14, C15, C16, C17, C18, C19, C2, C20, C21, C22, C23, C24, C25, C26, C27, C3, C31, C32, C33, C4, C5, C6, C7, C8: LCSC (none) -> C14663; MPN (none) -> CC0603KRX7R9BB104; Manufacturer (none) -> YAGEO
- C10, C13, C28, C29, C30, C9: LCSC (none) -> C15850; MPN (none) -> CL21A106KAYNNNE; Manufacturer (none) -> Samsung Electro-Mechanics
- C34, C36, C38, C40: LCSC (none) -> C15849; MPN (none) -> CL10A105KB8NNNC; Manufacturer (none) -> Samsung Electro-Mechanics
- C35: value 100nF -> 1uF; LCSC (none) -> C15849; MPN (none) -> CL10A105KB8NNNC; Manufacturer (none) -> Samsung Electro-Mechanics
- C37, C39: LCSC (none) -> C163508; MPN (none) -> CL10C102JB8NNNC; Manufacturer (none) -> Samsung Electro-Mechanics
- D1: value LED green 0603 -> LED yellow-green 0603; LCSC (none) -> C2986011; MPN (none) -> 19-21SYGC/S530-E2/4T; Manufacturer (none) -> Everlight
- R1: LCSC (none) -> C23140; MPN (none) -> 0603WAF330JT5E; Manufacturer (none) -> UNI-ROYAL
- R10, R11, R17, R24, R25, R27, R29, R31, R32, R33, R34, R35, R36, R37, R38, R39, R4, R40, R5: LCSC (none) -> C25804; MPN (none) -> 0603WAF1002T5E; Manufacturer (none) -> UNI-ROYAL
- R12, R13, R14, R22, R23, R3, R41, R6, R7, R8, R9: LCSC (none) -> C23162; MPN (none) -> 0603WAF4701T5E; Manufacturer (none) -> UNI-ROYAL
- R15: LCSC (none) -> C2999594; MPN (none) -> FRC0603F6493TS; Manufacturer (none) -> FOJAN
- R16: LCSC (none) -> C25803; MPN (none) -> 0603WAF1003T5E; Manufacturer (none) -> UNI-ROYAL
- R18, R2: LCSC (none) -> C21190; MPN (none) -> 0603WAF1001T5E; Manufacturer (none) -> UNI-ROYAL
- R26, R28, R30: LCSC (none) -> C4184; MPN (none) -> 0603WAF2002T5E; Manufacturer (none) -> UNI-ROYAL
- RT1: LCSC (none) -> C279936; MPN (none) -> SDNT1608X103F3950FTF; Manufacturer (none) -> Sunlord
- TP1, TP2, TP3, TP4, TP5: now left out of the parts list
- U1: Manufacturer (none) -> Lattice Semiconductor
- U2: Manufacturer (none) -> Winbond
- U3: Manufacturer (none) -> Texas Instruments
- U6: footprint Package_DFN_QFN:Texas_RTE0016D_WQFN-16-1EP_3x3mm_P0.5mm_EP0.8x0.8mm -> Package_DFN_QFN:WQFN-16-1EP_3x3mm_P0.5mm_EP1.68x1.68mm; Manufacturer (none) -> Texas Instruments; Note ADDR open: I2C address 0x10 (SBAS961A table 2: no resistor on ADDR; straight to ground is not a listed setting); AIN4 = FPGA_1V1 direct; footprint EP size to verify against SBAS961A mechanical drawing -> ADDR open: I2C address 0x10 (SBAS961A table 2: no resistor on ADDR; straight to ground is not a listed setting); AIN4 = FPGA_1V1 direct; exposed pad 1.68 x 1.68 mm as TI package RTE0016C (checked 2026-10-02)
- X1: Manufacturer (none) -> Interquip; Note CMOS 3.3 V, +-50 ppm, 10 mA (JLC stock 7439) -> CMOS 3.3 V, +-50 ppm, 10 mA; pad 1 enable (high), 2 ground,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
Connections:
- net FPGA_3V3: now also C46.1
- net GND: now also C46.2
Other:
- moved on the sheet: R22, R23, R24, R25, R26, R27, R28, R29, R30, R31, R32, RT1
