File: hardware/sn64-v2/power.kicad_sch (KiCad schematic)
At the start: 52 parts, among them J101 DX07S016JA3R1500, U10 TLV62569DBVR, U11 AP2112K-2.5TRG1, U12 TPS2553DBVR, U4 USBLC6-2SC6, U7 TPS2121RUXR, U8 TPS63070RNMR, U9 TLV62569DBVR

Commit message: Cartridge check: detect a reversed cartridge before 5 V is switched on
Owner idea (2026-10-01): detect a SNES cartridge that is in back to front and
say so on the screen. A reversed cartridge has its ground on the socket's 5 V
pins (contact k lands on 63 - k, checked on the footprint), so until now the
switch would push its 1.04 A limit backwards through it for up to 10 ms.

FPGA (v2 board, no added part): before the switch is enabled, the telemetry
ADC's channel 3 becomes a push-pull output so the divider's 20 k feeds at most
0.165 mA into the switched-off rail; the rail is read back about every 21 ms.
A reversed or shorted cartridge holds the rail low. New sequencer states 7-9,
fault code 0x01, /RESET released during the check. Modes in CONTROL bits 5:4:
enforce (reset default), report only, off, check only (never powers). Result
in the new CART_CHECK register at 0x0A. SEQ_PROBE_ENABLE = 0 leaves it out.

Boot menu: "Check cartridge (no power)", a "Cartridge check:" setting that
starts in report only until real cartridges have been measured, the last
result on the main screen, and an alert screen ("WHOA. WRONG WAY ROUND. ...").
The game display is now entered only once the cartridge really runs.

Evidence (simulation only): tb_cart_check (ADC model and electrical model of
the rail) and ten more cases in tb_power_sequencer, with fault-injected runs
that must fail; tb_n64_endpoint; host tests for the screens; the ROM builds
and passes its checks and its co-simulation; route_top --top board --speed 8
passes on all five clocks. The thresholds (0.65 V, 4 s) are assumptions;
nothing has been measured on a cartridge.

Also: the notes for U6 and U12 now cite the datasheets read today (SBAS961A,
SLVS841F) and give the 24.9 k current limit as computed (1.04 A nominal); the
ROM co-simulation script has its two missing source files back.

Co-Authored-By: Claude Opus 5.5 <noreply@anthropic.com>
Parts:
- U12: Note RILIM 24.9k ~ 1.0 A typ (provisional, SLVS963 equation to c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 -> RILIM 24.9k: 1.04 A nominal, 0.96 to 1.12 A (SLVS841F equat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
Changed lines of the file:
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@@
 (property "LCSC" "C55266" (at 67.31 360.68 0) (effects (font (size 1.27 1.27)) (hide yes)))
 (property "MPN" "TPS2553DBVR" (at 67.31 360.68 0) (effects (font (size 1.27 1.27)) (hide yes)))
-(property "Note" "RILIM 24.9k ~ 1.0 A typ (provisional, SLVS963 equation to confirm at review)" (at 67.31 360.68 0) (effects (font (size 1.27 1.27)) (hide yes)))
+(property "Note" "RILIM 24.9k: 1.04 A nominal, 0.96 to 1.12 A (SLVS841F equations, checked 2026-10-01)" (at 67.31 360.68 0) (effects (font (size 1.27 1.27)) (hide yes)))
 (pin "1")
 (pin "3")
