File: hardware/sn64-v2/power.kicad_sch (KiCad schematic)
At the start: 52 parts, among them J101 DX07S016JA3R1500, U10 TLV62569DBVR, U11 AP2112K-2.5TRG1, U12 TPS2553DBVR, U4 USBLC6-2SC6, U7 TPS2121RUXR, U8 TPS63070RNMR, U9 TLV62569DBVR

Commit message: USB loader chip (FT231X on JTAG), USB-C on the player's right, no USB logic in the FPGA; board copper complete
The owner: "Add back just the usb loader chip and put the usb on the right side of the cart",
and of the FPGA's own USB logic: "no i want it clean so remove it".

Board (hardware/sn64-v2)
- U13 FT231XS between the USB-C socket and the FPGA's JTAG port, wired like the ULX3S so that
  openFPGALoader drives it as it is (-b ulx3s): TCK on DSR#, TMS on DCD#, TDI on RI#, TDO on CTS#.
  Bus-powered as FTDI's data sheet draws it; with no cable it has no supply.
- Six small parts with it: three 100 nF, two 47 pF, and the 4.7 k pull-down on TCK that Lattice
  asks for. R19 and R20 are its 27 ohm series resistors now; R21 and R201 are gone. 182 parts.
- The socket, its protection part and the VBUS capacitor are on the -X edge, the player's right.
- apply_usb_loader_v2.py carries it into the routed board: 19 nets routed with everything else
  locked, a keep-out under the socket's body. VBUS to the input switch: 55 mm, was 104 mm.
- close_open_items_v2.py closes what KiCad's check still listed: the N64 controller line (a
  leftover via), the converter's 3.3 V pin, flash D2 at the corner of the ball grid (laid again
  together with its two neighbours) and five ground pads with a single thermal spoke (now solid).
  KiCad's rule check: no error, no open connection, 217 of 217 signal nets.
- Wiring check: 22 of 22; 25 of 25 deliberate mistakes caught, five of them new.

FPGA (fpga/)
- The USB device, its two clocks, its share of the flash and the reboot line are out of the
  logic, with the TinyFPGA core and the two tools that prepared it. The flash reader is
  SummerCart64's memory_flash unmodified again. 28,955 LUT4 (30,820 before), 107 pins (111),
  4 clocks (6).
- evaluate.py --mode sim passes; every clock passes on the board's pins.
- The game run of 660 pictures is the same as before, picture for picture, and the sound byte
  for byte.

Board-level runs on the new boa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
Parts:
- added C41, C42, C43: 100nF 16V X7R, Capacitor_SMD:C_0603_1608Metric, symbol Device:C
- added C44, C45: 47pF 50V C0G, Capacitor_SMD:C_0603_1608Metric, symbol Device:C
- added R19, R20: 27, Resistor_SMD:R_0603_1608Metric, symbol Device:R
- added U13: FT231XS-R, Package_SO:SSOP-20_3.9x8.7mm_P0.635mm, symbol Interface_USB:FT231XS
Connections:
- net GND: now also C41.2, C42.2, C43.2, C44.2, C45.2, U13.16 (GND), U13.6 (GND)
- net USB_DN: now also C45.1, R20.1
- net USB_DP: now also C44.1, R19.1
- net USB_VBUS: now also C41.1, U13.15 (VCC)
- new net FT_3V3: C42.1, C43.1, U13.13 (3V3OUT), U13.14 (~{RESET}), U13.3 (VCCIO)
- new net JTAG_TCK: U13.7 (~{DSR})
- new net JTAG_TDI: U13.5 (~{RI})
- new net JTAG_TDO: U13.9 (~{CTS})
- new net JTAG_TMS: U13.8 (~{DCD})
- new net USB_DN_F: R20.2, U13.12 (USBDM)
- new net USB_DP_F: R19.2, U13.11 (USBDP)
- no-connect marks 4 -> 12
Other:
- note added: "SN64 v2 POWER SHEET - TPS2121 input mux (USB priority) -> TPS63070 buck-boost 5V_SYS -> TLV62569 x2 (3V3, 1V1), AP2112K-2.5 LDO (2V5), TPS2553 cartridge switch, USB-C receptacle with the loader chip (FT231X on the FPGA JTAG port). Converter values are the v1 ones (verified pin tables)."
- note removed: "SN64 v2 POWER SHEET - TPS2121 input mux (USB priority) -> TPS63070 buck-boost 5V_SYS -> TLV62569 x2 (3V3, 1V1), AP2112K-2.5 LDO (2V5), TPS2553 cartridge switch, USB-C receptacle. Converter values are the v1 ones (verified pin tables)."
- moved on the sheet: C303, C304, C305, C306, C307, C308, C309, C310, C311, C312, C313, C314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

Commit message: Pre-order review, work in progress: finger fill, U6 footprint, USB-C port from the drawings, parts list numbers, power re-layout started
Checkpoint in the middle of the review, committed at the owner's request. Not a release.

Done and on the board file:
- ground fill taken out of the N64 edge fingers, ground plane extended to the finger vias
  (apply_finger_clearance_v2.py)
- U6 footprint with the exposed pad of its data sheet, R17 moved, leftovers of the first
  routing trimmed, silkscreen labels tidied, part records synced with the schematic
- USB supply capacitance 8.0 uF, selector soft-start 10 nF

Done elsewhere:
- shell: USB-C port from the JAE drawing, the USB-IF plug limits and the SummerCart64 port
- a maker part number on every bought part; yellow-green lamp; 1 uF at each ADC supply pin
- pack_bitstream.py: the FPGA image packed for a fast load, and the whole flash as one file
- make_production_v2.py (its output is not in this commit: it is remade when the board is done)

In progress, schematic ahead of the board:
- the schematic has 12 more small parts (R321, C324, C325, C213-C220, C46) that the makers'
  data sheets ask for; the board file does not have them yet
- apply_power_layout_v2.py and make_power_plan.py lay the power section out again by the
  makers' layout rules; so far only on working copies under build/

Co-Authored-By: Claude Opus 5.5 <noreply@anthropic.com>
Parts:
- added C324, C325: 10uF 25V, Capacitor_SMD:C_0603_1608Metric, symbol Device:C
- added R321: 10k, Resistor_SMD:R_0603_1608Metric, symbol Device:R
- C301: value 4.7uF 10V -> 2.2uF 10V; LCSC (none) -> C377773; MPN (none) -> CL21A225KBQNNNE; Manufacturer (none) -> Samsung Electro-Mechanics
- C302, C320: LCSC (none) -> C15849; MPN (none) -> CL10A105KB8NNNC; Manufacturer (none) -> Samsung Electro-Mechanics
- C303: value 1nF -> 10nF; LCSC (none) -> C57112; MPN (none) -> 0603B103K500NT; Manufacturer (none) -> FH (Fenghua)
- C304: value 10uF 10V -> 4.7uF 10V; LCSC (none) -> C1779; MPN (none) -> CL21A475KAQNNNE; Manufacturer (none) -> Samsung Electro-Mechanics
- C305, C306, C308, C323: LCSC (none) -> C15850; MPN (none) -> CL21A106KAYNNNE; Manufacturer (none) -> Samsung Electro-Mechanics
- C307, C322, C41, C42, C43: LCSC (none) -> C14663; MPN (none) -> CC0603KRX7R9BB104; Manufacturer (none) -> YAGEO
- C309, C310, C311, C312, C313, C316, C317, C318, C319: LCSC (none) -> C45783; MPN (none) -> CL21A226MAQNNNE; Manufacturer (none) -> Samsung Electro-Mechanics
- C314, C315: LCSC (none) -> C1679; MPN (none) -> 0603CG6R8C500NT; Manufacturer (none) -> FH (Fenghua)
- C321: LCSC (none) -> C1779; MPN (none) -> CL21A475KAQNNNE; Manufacturer (none) -> Samsung Electro-Mechanics
- C44, C45: LCSC (none) -> C1671; MPN (none) -> CL10C470JB8NNNC; Manufacturer (none) -> Samsung Electro-Mechanics
- J101: Manufacturer (none) -> JAE
- L1: Manufacturer (none) -> APV
- L2, L3: Manufacturer (none) -> Changjiang Microelectronics
- R19, R20: LCSC (none) -> C25190; MPN (none) -> 0603WAF270JT5E; Manufacturer (none) -> UNI-ROYAL
- R301, R302: LCSC (none) -> C23186; MPN (none) -> 0603WAF5101T5E; Manufacturer (none) -> UNI-ROYAL
- R303: LCSC (none) -> C5126128; MPN (none) -> FRC0603F2743TS; Manufacturer (none) -> FOJAN
- R304, R306, R311, R319: LCSC (none) -> C25803; MPN (none) -> 0603WAF1003T5E; Manufacturer (none) -> UNI-ROYAL
- R305: LCSC (none) -> C5126102; MPN (none) -> FRC0603F1823TS; Manufacturer (none) -> FOJAN
- R307: LCSC (none) -> C2930103; MPN (none) -> FRC0603F4422TS; Manufacturer (none) -> FOJAN
- R308, R320: LCSC (none) -> C25804; MPN (none) -> 0603WAF1002T5E; Manufacturer (none) -> UNI-ROYAL
- R309: LCSC (none) -> C861240; MPN (none) -> RT0603BRD07232KL; Manufacturer (none) -> YAGEO
- R310: LCSC (none) -> C861410; MPN (none) -> RT0603BRD0744K2L; Manufacturer (none) -> YAGEO
- R312: LCSC (none) -> C6288321; MPN (none) -> RT0603BRD07459KL; Manufacturer (none) -> YAGEO
- R313: LCSC (none) -> C861068; MPN (none) -> RT0603BRD07102KL; Manufacturer (none) -> YAGEO
- R315: LCSC (none) -> C122538; MPN (none) -> RT0603BRD07100KL; Manufacturer (none) -> YAGEO
- R316: LCSC (none) -> C705720; MPN (none) -> RT0603BRD07120KL; Manufacturer (none) -> YAGEO
- R318: LCSC (none) -> C25962; MPN (none) -> 0603WAF2492T5E; Manufacturer (none) -> UNI-ROYAL
- U10, U12, U7, U8, U9: Manufacturer (none) -> Texas Instruments
- U11: Manufacturer (none) -> Diodes Incorporated
- U13: Manufacturer (none) -> FTDI
- U4: Manufacturer (none) -> STMicroelectronics
Connections:
- net 5V_SYS: now also C325.1
- net GND: now also C324.2, C325.2
- net SYS_VIN: now also C324.1, R321.1; no longer U8.14 (EN)
- new net EN_5V: R321.2, U8.14 (EN)
Other:
- moved on the sheet: C307, C308, C309, C310, C311, C312, C313
