File: hardware/sn64-v2/sn64-v2.kicad_pcb (KiCad board)
At the start: 6 copper layers, 111 x 70.5 mm, 182 parts, among them J1 N64 cartridge edge, J101 DX07S016JA3R1500, J2 SNES cartridge socket 62, U1 LFE5U-85F-8BG381I, U10 TLV62569DBVR, U11 AP2112K-2.5TRG1, U12 TPS2553DBVR, U2 W25Q128JVSIQ, U201 SN74ALVC164245DGGR, U202 SN74ALVC164245DGGR, U203 SN74ALVC164245DGGR, U204 SN74ALVC164245DGGR, U205 SN74LVC07APWR, U3 TPS3808G01DBVR, U4 USBLC6-2SC6, U6 TLA2528IRTER, U7 TPS2121RUXR, U8 TPS63070RNMR, U9 TLV62569DBVR, X1 27MHz 1631-27005-BTBEYA

Commit message: Board posts that pass through the board, registration pins, 4.0 mm board holes
The owner wants the board mounted the way a Nintendo cartridge mounts its board, not pinched
between two flat post ends, and wants it impossible to put the board in backward.

- Shell: at H1, H2, H5 and H6 the label-side post has a shelf and a hollow through-hole
  section 3.8 mm across and 1.1 mm high; the back post lands on the board and holds it on
  the shelf. The screw runs through both and cuts thread only below the shelf.
- Board: H1, H2, H5 and H6 are 4.0 mm so the hollow post fits (set_mounting_holes_v2.py).
  No copper within 4.5 mm; zones refilled; checks unchanged (6 starved thermals, 6 open
  items). Renders, copper picture and STEP regenerated.
- Registration: two solid pins through H3 and H4, at different heights left and right. The
  real board model turned back to front is stopped at both pins and the back half cannot
  close over it.
- finish_route_v2.py --refill-only: the pour removal breaks KiCad 10 python on a board that
  already has pours.

Checked in CAD only; hole sizes for M2 screws are assumptions.

Co-Authored-By: Claude Opus 5.5 <noreply@anthropic.com>
Parts:
- H1, H2, H5, H6: value MountingHole_2.5mm -> MountingHole_4mm; footprint MountingHole_2.5mm -> MountingHole:MountingHole_4mm

Commit message: A game through the board's own wiring; two wiring rules corrected from the data sheets
The owner's game now runs through a model of the v2 board that is generated
from the board file: the real top level on its balls, a model of every part on
its pads with the makers' pin numbers, the cartridge on the socket's pins and
the N64 on the edge fingers (make_board_sim.py, tb_board_game.sv,
run_game.py --board).

Found by reading each maker's data sheet, corrected on the board:
- U204's socket-to-FPGA byte was enabled all the time, also while its 5 V side
  has no supply. It now has an enable of its own (SENSE_OE_N, R214).
- The supply converter's address pin was tied to ground; the sheet gives the
  address the logic uses for the pin left open.

Found by the board run, corrected in the logic:
- the status LED was dark in a game;
- the cartridge's pins were loose for a moment at start and at power-off. They
  are now held at rest while the cartridge has its 5 V, and /RESET is held 1 ms
  before the 5 V goes.

Wiring check 21 of 21, 20 of 20 deliberate mistakes caught. The board run
refuses a reversed cartridge and two deliberately mis-wired boards. The logic
suite passes with two new fault builds; the design routes with every clock
passing. Test set results: 38 of 38 judged programs pass.

Still open before an order: six unrouted connections, the socket sample, the
first load of a blank board (docs/design/board-verification.md).

Co-Authored-By: Claude Opus 5.5 <noreply@anthropic.com>
Parts:
- added R214: 100k, R_0603_1608Metric, B.Cu at (-39.0, -41.9)
Connections:
- J1 pad 13: (no net) -> unconnected-(J1-12V-Pad13)
- J1 pad 14: (no net) -> unconnected-(J1-KEY1_RESERVED-Pad14)
- J1 pad 24: (no net) -> unconnected-(J1-AUDIO_L-Pad24)
- J1 pad 38: (no net) -> unconnected-(J1-12V-Pad38)
- J1 pad 39: (no net) -> unconnected-(J1-KEY2_RESERVED-Pad39)
- J1 pad 46: (no net) -> unconnected-(J1-VIDEO_SYNC_RESERVED-Pad46)
- J1 pad 49: (no net) -> unconnected-(J1-AUDIO_R-Pad49)
- U1 pad U19: L_EXPAND -> SENSE_OE_N
- U204 pad 19: SNES_EXPAND -> GND
- U204 pad 25: GND -> SENSE_OE_N
- U204 pad 26: unconnected-(U204-2A7-Pad26) -> GND
- U204 pad 27: unconnected-(U204-2A6-Pad27) -> GND
- U204 pad 29: unconnected-(U204-2A5-Pad29) -> GND
- U204 pad 30: L_EXPAND -> GND
- U6 pad 11: GND -> unconnected-(U6-ADDR-Pad11)
Routing:
- net SENSE_OE_N: track 0.00 -> 66.0 mm, vias 0 -> 4
- net L_EXPAND: track 62.2 -> 0.00 mm, vias 4 -> 0
- net SNES_EXPAND: track 93.8 -> 47.2 mm, vias 8 -> 2
- net FPGA_3V3: track 104.7 -> 106.2 mm
- net GND: track 306.7 -> 307.2 mm, vias 265 -> 264
