File: hardware/sn64-v2/cart.kicad_sch (KiCad schematic)
At the start: 32 parts, among them J1 Riser joint 2x20 2.00mm, J2 SNES cartridge socket 62, U201 SN74ALVC164245DGGR, U202 SN74ALVC164245DGGR, U203 SN74ALVC164245DGGR, U204 SN74ALVC164245DGGR, U205 SN74LVC07APWR

Commit message: v2 single board: routed board, schematic with the N64 edge, validation reports, renders and notes
Co-Authored-By: Claude Fable 5.1 <noreply@anthropic.com>
Parts:
- J1: value Riser joint 2x20 2.00mm -> N64 cartridge edge; footprint Connector_PinSocket_2.00mm:PinSocket_2x20_P2.00mm_Vertical -> SN64:N64_Edge_SC64_Reference; symbol Connector_Generic:Conn_02x20_Odd_Even -> SN64:N64_Cartridge_Edge_50; Note pins 1-27 N64 bus, 28-31 HOST_3V3, 32-40 GND; mates hardwar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 -> SummerCart64 edge geometry; 12 V, audio, sync and key finge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
Connections:
- net GND: now also J1.1 (GND), J1.2 (GND), J1.22 (GND), J1.23 (GND), J1.25 (GND), J1.26 (GND), J1.27 (GND), J1.31 (GND), J1.47 (GND), J1.48 (GND), J1.50 (GND), J1.6 (GND); no longer J1.32 (Pin_32), J1.33 (Pin_33), J1.34 (Pin_34), J1.35 (Pin_35), J1.36 (Pin_36), J1.37 (Pin_37), J1.38 (Pin_38), J1.39 (Pin_39), J1.40 (Pin_40)
- net HOST_3V3: now also J1.17 (3V3), J1.34 (3V3), J1.42 (3V3), J1.9 (3V3); no longer J1.28 (Pin_28), J1.29 (Pin_29), J1.30 (Pin_30), J1.31 (Pin_31)
- net N64_AD0: now also J1.28 (AD0); no longer J1.1 (Pin_1)
- net N64_AD1: now also J1.29 (AD1); no longer J1.2 (Pin_2)
- net N64_AD10: now also J1.12 (AD10); no longer J1.11 (Pin_11)
- net N64_AD11: now also J1.11 (AD11); no longer J1.12 (Pin_12)
- net N64_AD12: now also J1.7 (AD12); no longer J1.13 (Pin_13)
- net N64_AD13: now also J1.5 (AD13); no longer J1.14 (Pin_14)
- net N64_AD14: now also J1.4 (AD14); no longer J1.15 (Pin_15)
- net N64_AD15: now also J1.3 (AD15); no longer J1.16 (Pin_16)
- net N64_AD2: now also J1.30 (AD2); no longer J1.3 (Pin_3)
- net N64_AD3: now also J1.32 (AD3); no longer J1.4 (Pin_4)
- net N64_AD4: now also J1.36 (AD4); no longer J1.5 (Pin_5)
- net N64_AD5: now also J1.37 (AD5); no longer J1.6 (Pin_6)
- net N64_AD6: now also J1.40 (AD6); no longer J1.7 (Pin_7)
- net N64_AD7: now also J1.41 (AD7); no longer J1.8 (Pin_8)
- net N64_AD8: now also J1.16 (AD8); no longer J1.9 (Pin_9)
- net N64_AD9: now also J1.15 (AD9); no longer J1.10 (Pin_10)
- net N64_ALE_H: now also J1.35 (ALE_H); no longer J1.18 (Pin_18)
- net N64_ALE_L: now also J1.33 (ALE_L); no longer J1.17 (Pin_17)
- net N64_CIC_CLK: now also J1.43 (CIC_CLK); no longer J1.24 (Pin_24)
- net N64_CIC_DATA: now also J1.18 (CIC_DATA); no longer J1.25 (Pin_25)
- net N64_INT_N: now also J1.44 (/INT); no longer J1.23 (Pin_23)
- net N64_JOYBUS: now also J1.21 (JOYBUS); no longer J1.27 (Pin_27)
- net N64_NMI_N: now also J1.45 (/NMI); no longer J1.22 (Pin_22)
- net N64_PIF_CLK: now also J1.19 (PIF_CLK); no longer J1.26 (Pin_26)
- net N64_READ_N: now also J1.10 (/READ); no longer J1.19 (Pin_19)
- net N64_RESET_N: now also J1.20 (/RESET); no longer J1.21 (Pin_21)
- net N64_WRITE_N: now also J1.8 (/WRITE); no longer J1.20 (Pin_20)
- no-connect marks 10 -> 17
Other:
- note added: "SN64 v2 CARTRIDGE SHEET - N64 edge J1 and SNES socket J2 on the one board, four SN74ALVC164245 translators (A = 3.3 V, B = 5 V), SN74LVC07A open-drain driver for the 5 V lines the FPGA pulls."
- note removed: "SN64 v2 CARTRIDGE SHEET - SNES socket J2 on this board (no joint), four SN74ALVC164245 translators (A = 3.3 V, B = 5 V), SN74LVC07A open-drain driver for the 5 V lines the FPGA pulls."
- moved on the sheet: C212

Commit message: v2 board refitted to the tower shell: SNES socket straddling the top edge, USB-C above the console
- New footprint SN64_V2:SNES_Slot_Console_Straddle (pins 1-31 on B.Cu, the face toward the
  front of the console; 32-62 on F.Cu) with a 3D model of the eared socket; generator and
  schematic point J2 at it (schematic diff: J2 footprint and note only).
- refit_tower_v2.py: clear (old socket, copper above the translators, USB-C nets cut at the
  old connector, dangling trim), place (outline 111 mm at the USB-C, 88 mm neck, J2 on the
  top edge, USB-C + ESD + VBUS cap at 50 mm, holes moved, planes enlarged, existing copper
  locked), unlock. KiCadRoutingTools routed 64/64 nets with nothing broken.
- DRC (board rules): 5 single-spoke thermal reliefs, 6 known open items; ERC unchanged.
- Fit check: the KiCad STEP with all part models has no interference with the shell.

Co-Authored-By: Claude Opus 5.5 <noreply@anthropic.com>
Parts:
- J2: footprint SN64:SNES_Slot_Console_7mm -> SN64_V2:SNES_Slot_Console_Straddle; Note candidate NES Repair Shop snspt043; footprint from Sanni ca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 -> console-replacement socket with ears (sample candidate NES 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
Changed lines of the file:
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@@
 (property "Reference" "J2" (at 49.53 46.99 0) (effects (font (size 1.27 1.27)) (justify left)))
 (property "Value" "SNES cartridge socket 62" (at 49.53 49.53 0) (effects (font (size 1.27 1.27)) (justify left)))
-(property "Footprint" "SN64:SNES_Slot_Console_7mm" (at 92.71 130.81 0) (effects (font (size 1.27 1.27)) (hide yes)))
+(property "Footprint" "SN64_V2:SNES_Slot_Console_Straddle" (at 92.71 130.81 0) (effects (font (size 1.27 1.27)) (hide yes)))
 (property "Datasheet" "" (at 92.71 130.81 0) (effects (font (size 1.27 1.27)) (hide yes)))
-(property "Note" "candidate NES Repair Shop snspt043; footprint from Sanni cartreader (CC-BY-4.0), 7 mm nose" (at 92.71 130.81 0) (effects (font (size 1.27 1.27)) (hide yes)))
+(property "Note" "console-replacement socket with ears (sample candidate NES Repair Shop snspt043); straddles the board top edge, pins 1-31 on B.Cu (front of the console); ears screw to the shell; pin geometry from OpenSFC CartSlot" (at 92.71 130.81 0) (effects (font (size 1.27 1.27)) (hide yes)))
 (pin "1")
 (pin "2")

Commit message: A game through the board's own wiring; two wiring rules corrected from the data sheets
The owner's game now runs through a model of the v2 board that is generated
from the board file: the real top level on its balls, a model of every part on
its pads with the makers' pin numbers, the cartridge on the socket's pins and
the N64 on the edge fingers (make_board_sim.py, tb_board_game.sv,
run_game.py --board).

Found by reading each maker's data sheet, corrected on the board:
- U204's socket-to-FPGA byte was enabled all the time, also while its 5 V side
  has no supply. It now has an enable of its own (SENSE_OE_N, R214).
- The supply converter's address pin was tied to ground; the sheet gives the
  address the logic uses for the pin left open.

Found by the board run, corrected in the logic:
- the status LED was dark in a game;
- the cartridge's pins were loose for a moment at start and at power-off. They
  are now held at rest while the cartridge has its 5 V, and /RESET is held 1 ms
  before the 5 V goes.

Wiring check 21 of 21, 20 of 20 deliberate mistakes caught. The board run
refuses a reversed cartridge and two deliberately mis-wired boards. The logic
suite passes with two new fault builds; the design routes with every clock
passing. Test set results: 38 of 38 judged programs pass.

Still open before an order: six unrouted connections, the socket sample, the
first load of a blank board (docs/design/board-verification.md).

Co-Authored-By: Claude Opus 5.5 <noreply@anthropic.com>
Parts:
- added R214: 100k, Resistor_SMD:R_0603_1608Metric, symbol Device:R
Connections:
- net L_EXPAND is gone; now on net GND: U204.30 (2A4)
- net FPGA_3V3: now also R214.1
- net GND: now also U204.19 (2B4), U204.26 (2A7), U204.27 (2A6), U204.29 (2A5); no longer U204.25 (2~{OE})
- net SNES_EXPAND: no longer U204.19 (2B4)
- new net SENSE_OE_N: R214.2, U204.25 (2~{OE})
- no-connect marks 17 -> 14
Changed lines of the file:
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@@
 (global_label "SNES_RESET_N" (shape passive) (at 300.99 288.29 180) (fields_autoplaced yes) (effects (font (size 1.016 1.016)) (justify right)) (property "Intersheetrefs" "${INTERSHEET_REFS}" (at 300.99 288.29 0) (effects (font (size 1.27 1.27)) (hide yes))))
 (wire (pts (xy 306.07 290.83) (xy 300.99 290.83)) (stroke (width 0) (type default)))
-(global_label "SNES_EXPAND" (shape passive) (at 300.99 290.83 180) (fields_autoplaced yes) (effects (font (size 1.016 1.016)) (justify right)) (property "Intersheetrefs" "${INTERSHEET_REFS}" (at 300.99 290.83 0) (effects (font (size 1.27 1.27)) (hide yes))))
+(global_label "GND" (shape passive) (at 300.99 290.83 180) (fields_autoplaced yes) (effects (font (size 1.016 1.016)) (justify right)) (property "Intersheetrefs" "${INTERSHEET_REFS}" (at 300.99 290.83 0) (effects (font (size 1.27 1.27)) (hide yes))))
 (wire (pts (xy 306.07 293.37) (xy 300.99 293.37)) (stroke (width 0) (type default)))
 (global_label "GND" (shape passive) (at 300.99 293.37 180) (fields_autoplaced yes) (effects (font (size 1.016 1.016)) (justify right)) (property "Intersheetrefs" "${INTERSHEET_REFS}" (at 300.99 293.37 0) (effects (font (size 1.27 1.27)) (hide yes))))
@@
 (global_label "GND" (shape passive) (at 300.99 255.27 180) (fields_autoplaced yes) (effects (font (size 1.016 1.016)) (justify right)) (property "Intersheetrefs" "${INTERSHEET_REFS}" (at 300.99 255.27 0) (effects (font (size 1.27 1.27)) (hide yes))))
 (wire (pts (xy 331.47 255.27) (xy 336.55 255.27)) (stroke (width 0) (type default)))
-(global_label "GND" (shape passive) (at 336.55 255.27 0) (fields_autoplaced yes) (effects (font (size 1.016 1.016)) (justify left)) (property "Intersheetrefs" "${INTERSHEET_REFS}" (at 336.55 255.27 0) (effects (font (size 1.27 1.27)) (hide yes))))
-(no_connect (at 331.47 298.45))
-(no_connect (at 331.47 295.91))
-(no_connect (at 331.47 293.37))
+(global_label "SENSE_OE_N" (shape passive) (at 336.55 255.27 0) (fields_autoplaced yes) (effects (font (size 1.016 1.016)) (justify left)) (property "Intersheetrefs" "${INTERSHEET_REFS}" (at 336.55 255.27 0) (effects (font (size 1.27 1.27)) (hide yes))))
+(wire (pts (xy 331.47 298.45) (xy 336.55 298.45)) (stroke (width 0) (type default)))
+(global_label "GND" (shape passive) (at 336.55 298.45 0) (fields_autoplaced yes) (effects (font (size 1.016 1.016)) (justify left)) (property "Intersheetrefs" "${INTERSHEET_REFS}" (at 336.55 298.45 0) (effects (font (size 1.27 1.27)) (hide yes))))
+(wire (pts (xy 331.47 295.91) (xy 336.55 295.91)) (stroke (width 0) (type default)))
+(global_label "GND" (shape passive) (at 336.55 295.91 0) (fields_autoplaced yes) (effects (font (size 1.016 1.016)) (justify left)) (property "Intersheetrefs" "${INTERSHEET_REFS}" (at 336.55 295.91 0) (effects (font (size 1.27 1.27)) (hide yes))))
+(wire (pts (xy 331.47 293.37) (xy 336.55 293.37)) (stroke (width 0) (type default)))
+(global_label "GND" (shape passive) (at 336.55 293.37 0) (fields_autoplaced yes) (effects (font (size 1.016 1.016)) (justify left)) (property "Intersheetrefs" "${INTERSHEET_REFS}" (at 336.55 293.37 0) (effects (font (size 1.27 1.27)) (hide yes))))
 (wire (pts (xy 331.47 290.83) (xy 336.55 290.83)) (stroke (width 0) (type default)))
-(global_label "L_EXPAND" (shape passive) (at 336.55 290.83 0) (fields_autoplaced yes) (effects (font (size 1.016 1.016)) (justify left)) (property "Intersheetrefs" "${INTERSHEET_REFS}" (at 336.55 290.83 0) (effects (font (size 1.27 1.27)) (hide yes))))
+(global_label "GND" (shape passive) (at 336.55 290.83 0) (fields_autoplaced yes) (effects (font (size 1.016 1.016)) (justify left)) (property "Intersheetrefs" "${INTERSHEET_REFS}" (at 336.55 290.83 0) (effects (font (size 1.27 1.27)) (hide yes))))
 (wire (pts (xy 321.31 242.57) (xy 321.31 237.49)) (stroke (width 0) (type default)))
 (global_label "FPGA_3V3" (shape passive) (at 321.31 237.49 90) (fields_autoplaced yes) (effects (font (size 1.016 1.016)) (justify left)) (property "Intersheetrefs" "${INTERSHEET_REFS}" (at 321.31 237.49 0) (effects (font (size 1.27 1.27)) (hide yes))))
@@
 (wire (pts (xy 156.21 441.96) (xy 156.21 447.04)) (stroke (width 0) (type default)))
 (global_label "DATA_DIR" (shape passive) (at 156.21 447.04 270) (fields_autoplaced yes) (effects (font (size 1.016 1.016)) (justify right)) (property "Intersheetrefs" "${INTERSHEET_REFS}" (at 156.21 447.04 0) (effects (font (size 1.27 1.27)) (hide yes))))
+(symbol (lib_id "Device:R") (at 171.45 438.15 0) (unit 1) (exclude_from_sim no) (in_bom yes) (on_board yes) (dnp no)
+(property "Reference" "R214" (at 173.99 436.88 0) (effects (font (size 1.27 1.27)) (justify left)))
+(property "Value" "100k" (at 173.99 439.42 0) (effects (font (size 1.27 1.27)) (justify left)))
+(property "Footprint" "Resistor_SMD:R_0603_1608Metric" (at 171.45 438.15 0) (effects (font (size 1.27 1.27)) (hide yes)))
+(property "Datasheet" "" (at 171.45 438.15 0) (effects (font (size 1.27 1.27)) (hide yes)))
+(pin "1")
+(pin "2")
+(instances (project "sn64-v2" (path "/d28f46aa-91c7-5060-a563-bf74d208e51e/69e05daa-4082-5d3e-8a2d-0d56f4a78932" (reference "R214") (unit 1)))))
+(wire (pts (xy 171.45 434.34) (xy 171.45 429.26)) (stroke (width 0) (type default)))
+(global_label "FPGA_3V3" (shape passive) (at 171.45 429.26 90) (fields_autoplaced yes) (effects (font (size 1.016 1.016)) (justify left)) (property "Intersheetrefs" "${INTERSHEET_REFS}" (at 171.45 429.26 0) (effects (font (size 1.27 1.27)) (hide yes))))
+(wire (pts (xy 171.45 441.96) (xy 171.45 447.04)) (stroke (width 0) (type default)))
+(global_label "SENSE_OE_N" (shape passive) (at 171.45 447.04 270) (fields_autoplaced yes) (effects (font (size 1.016 1.016)) (justify right)) (property "Intersheetrefs" "${INTERSHEET_REFS}" (at 171.45 447.04 0) (effects (font (size 1.27 1.27)) (hide yes))))
 (symbol (lib_id "SN64:N64_Cartridge_Edge_50") (at 92.71 542.29 0) (unit 1) (exclude_from_sim no) (in_bom yes) (on_board yes) (dnp no)
 (property "Reference" "J1" (at 49.53 473.71 0) (effects (font (size 1.27 1.27)) (justify left)))
