File: hardware/sn64-v2/cart.kicad_sch (KiCad schematic)
At the start: 33 parts, among them J1 N64 cartridge edge, J2 SNES cartridge socket 62, U201 SN74ALVC164245DGGR, U202 SN74ALVC164245DGGR, U203 SN74ALVC164245DGGR, U204 SN74ALVC164245DGGR, U205 SN74LVC07APWR

Commit message: USB loader chip (FT231X on JTAG), USB-C on the player's right, no USB logic in the FPGA; board copper complete
The owner: "Add back just the usb loader chip and put the usb on the right side of the cart",
and of the FPGA's own USB logic: "no i want it clean so remove it".

Board (hardware/sn64-v2)
- U13 FT231XS between the USB-C socket and the FPGA's JTAG port, wired like the ULX3S so that
  openFPGALoader drives it as it is (-b ulx3s): TCK on DSR#, TMS on DCD#, TDI on RI#, TDO on CTS#.
  Bus-powered as FTDI's data sheet draws it; with no cable it has no supply.
- Six small parts with it: three 100 nF, two 47 pF, and the 4.7 k pull-down on TCK that Lattice
  asks for. R19 and R20 are its 27 ohm series resistors now; R21 and R201 are gone. 182 parts.
- The socket, its protection part and the VBUS capacitor are on the -X edge, the player's right.
- apply_usb_loader_v2.py carries it into the routed board: 19 nets routed with everything else
  locked, a keep-out under the socket's body. VBUS to the input switch: 55 mm, was 104 mm.
- close_open_items_v2.py closes what KiCad's check still listed: the N64 controller line (a
  leftover via), the converter's 3.3 V pin, flash D2 at the corner of the ball grid (laid again
  together with its two neighbours) and five ground pads with a single thermal spoke (now solid).
  KiCad's rule check: no error, no open connection, 217 of 217 signal nets.
- Wiring check: 22 of 22; 25 of 25 deliberate mistakes caught, five of them new.

FPGA (fpga/)
- The USB device, its two clocks, its share of the flash and the reboot line are out of the
  logic, with the TinyFPGA core and the two tools that prepared it. The flash reader is
  SummerCart64's memory_flash unmodified again. 28,955 LUT4 (30,820 before), 107 pins (111),
  4 clocks (6).
- evaluate.py --mode sim passes; every clock passes on the board's pins.
- The game run of 660 pictures is the same as before, picture for picture, and the sound byte
  for byte.

Board-level runs on the new boa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
Parts:
- removed R201: 10k, Resistor_SMD:R_0603_1608Metric, symbol Device:R
Connections:
- net PROGRAMN_PULL is gone; now on net GND: U205.1
- net FPGA_PROGRAMN: no longer names the net of U205.2
- no-connect marks 14 -> 15
Other:
- moved on the sheet: R202, R203, R204
Changed lines of the file:
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@@
 (instances (project "sn64-v2" (path "/d28f46aa-91c7-5060-a563-bf74d208e51e/69e05daa-4082-5d3e-8a2d-0d56f4a78932" (reference "U205") (unit 1)))))
 (wire (pts (xy 49.53 379.73) (xy 44.45 379.73)) (stroke (width 0) (type default)))
-(global_label "PROGRAMN_PULL" (shape passive) (at 44.45 379.73 180) (fields_autoplaced yes) (effects (font (size 1.016 1.016)) (justify right)) (property "Intersheetrefs" "${INTERSHEET_REFS}" (at 44.45 379.73 0) (effects (font (size 1.27 1.27)) (hide yes))))
-(wire (pts (xy 64.77 379.73) (xy 69.85 379.73)) (stroke (width 0) (type default)))
-(global_label "FPGA_PROGRAMN" (shape passive) (at 69.85 379.73 0) (fields_autoplaced yes) (effects (font (size 1.016 1.016)) (justify left)) (property "Intersheetrefs" "${INTERSHEET_REFS}" (at 69.85 379.73 0) (effects (font (size 1.27 1.27)) (hide yes))))
+(global_label "GND" (shape passive) (at 44.45 379.73 180) (fields_autoplaced yes) (effects (font (size 1.016 1.016)) (justify right)) (property "Intersheetrefs" "${INTERSHEET_REFS}" (at 44.45 379.73 0) (effects (font (size 1.27 1.27)) (hide yes))))
+(no_connect (at 64.77 379.73))
 (symbol (lib_id "74xx:74LS07") (at 133.35 379.73 0) (unit 2) (exclude_from_sim no) (in_bom yes) (on_board yes) (dnp no)
 (property "Reference" "U205" (at 125.73 372.11 0) (effects (font (size 1.27 1.27)) (justify left)))
@@
 (global_label "GND" (shape passive) (at 539.75 386.08 270) (fields_autoplaced yes) (effects (font (size 1.016 1.016)) (justify right)) (property "Intersheetrefs" "${INTERSHEET_REFS}" (at 539.75 386.08 0) (effects (font (size 1.27 1.27)) (hide yes))))
 (symbol (lib_id "Device:R") (at 554.99 377.19 0) (unit 1) (exclude_from_sim no) (in_bom yes) (on_board yes) (dnp no)
-(property "Reference" "R201" (at 557.53 375.92 0) (effects (font (size 1.27 1.27)) (justify left)))
+(property "Reference" "R202" (at 557.53 375.92 0) (effects (font (size 1.27 1.27)) (justify left)))
 (property "Value" "10k" (at 557.53 378.46 0) (effects (font (size 1.27 1.27)) (justify left)))
 (property "Footprint" "Resistor_SMD:R_0603_1608Metric" (at 554.99 377.19 0) (effects (font (size 1.27 1.27)) (hide yes)))
@@
 (pin "1")
 (pin "2")
-(instances (project "sn64-v2" (path "/d28f46aa-91c7-5060-a563-bf74d208e51e/69e05daa-4082-5d3e-8a2d-0d56f4a78932" (reference "R201") (unit 1)))))
+(instances (project "sn64-v2" (path "/d28f46aa-91c7-5060-a563-bf74d208e51e/69e05daa-4082-5d3e-8a2d-0d56f4a78932" (reference "R202") (unit 1)))))
 (wire (pts (xy 554.99 373.38) (xy 554.99 368.3)) (stroke (width 0) (type default)))
 (global_label "FPGA_3V3" (shape passive) (at 554.99 368.3 90) (fields_autoplaced yes) (effects (font (size 1.016 1.016)) (justify left)) (property "Intersheetrefs" "${INTERSHEET_REFS}" (at 554.99 368.3 0) (effects (font (size 1.27 1.27)) (hide yes))))
 (wire (pts (xy 554.99 381) (xy 554.99 386.08)) (stroke (width 0) (type default)))
-(global_label "PROGRAMN_PULL" (shape passive) (at 554.99 386.08 270) (fields_autoplaced yes) (effects (font (size 1.016 1.016)) (justify right)) (property "Intersheetrefs" "${INTERSHEET_REFS}" (at 554.99 386.08 0) (effects (font (size 1.27 1.27)) (hide yes))))
+(global_label "CIC_DATA0_OD" (shape passive) (at 554.99 386.08 270) (fields_autoplaced yes) (effects (font (size 1.016 1.016)) (justify right)) (property "Intersheetrefs" "${INTERSHEET_REFS}" (at 554.99 386.08 0) (effects (font (size 1.27 1.27)) (hide yes))))
 (symbol (lib_id "Device:R") (at 571.5 377.19 0) (unit 1) (exclude_from_sim no) (in_bom yes) (on_board yes) (dnp no)
-(property "Reference" "R202" (at 574.04 375.92 0) (effects (font (size 1.27 1.27)) (justify left)))
+(property "Reference" "R203" (at 574.04 375.92 0) (effects (font (size 1.27 1.27)) (justify left)))
 (property "Value" "10k" (at 574.04 378.46 0) (effects (font (size 1.27 1.27)) (justify left)))
 (property "Footprint" "Resistor_SMD:R_0603_1608Metric" (at 571.5 377.19 0) (effects (font (size 1.27 1.27)) (hide yes)))
@@
 (pin "1")
 (pin "2")
-(instances (project "sn64-v2" (path "/d28f46aa-91c7-5060-a563-bf74d208e51e/69e05daa-4082-5d3e-8a2d-0d56f4a78932" (reference "R202") (unit 1)))))
+(instances (project "sn64-v2" (path "/d28f46aa-91c7-5060-a563-bf74d208e51e/69e05daa-4082-5d3e-8a2d-0d56f4a78932" (reference "R203") (unit 1)))))
 (wire (pts (xy 571.5 373.38) (xy 571.5 368.3)) (stroke (width 0) (type default)))
 (global_label "FPGA_3V3" (shape passive) (at 571.5 368.3 90) (fields_autoplaced yes) (effects (font (size 1.016 1.016)) (justify left)) (property "Intersheetrefs" "${INTERSHEET_REFS}" (at 571.5 368.3 0) (effects (font (size 1.27 1.27)) (hide yes))))
 (wire (pts (xy 571.5 381) (xy 571.5 386.08)) (stroke (width 0) (type default)))
-(global_label "CIC_DATA0_OD" (shape passive) (at 571.5 386.08 270) (fields_autoplaced yes) (effects (font (size 1.016 1.016)) (justify right)) (property "Intersheetrefs" "${INTERSHEET_REFS}" (at 571.5 386.08 0) (effects (font (size 1.27 1.27)) (hide yes))))
+(global_label "CIC_DATA1_OD" (shape passive) (at 571.5 386.08 270) (fields_autoplaced yes) (effects (font (size 1.016 1.016)) (justify right)) (property "Intersheetrefs" "${INTERSHEET_REFS}" (at 571.5 386.08 0) (effects (font (size 1.27 1.27)) (hide yes))))
 (symbol (lib_id "Device:R") (at 588.01 377.19 0) (unit 1) (exclude_from_sim no) (in_bom yes) (on_board yes) (dnp no)
-(property "Reference" "R203" (at 590.55 375.92 0) (effects (font (size 1.27 1.27)) (justify left)))
+(property "Reference" "R204" (at 590.55 375.92 0) (effects (font (size 1.27 1.27)) (justify left)))
 (property "Value" "10k" (at 590.55 378.46 0) (effects (font (size 1.27 1.27)) (justify left)))
 (property "Footprint" "Resistor_SMD:R_0603_1608Metric" (at 588.01 377.19 0) (effects (font (size 1.27 1.27)) (hide yes)))
@@
 (pin "1")
 (pin "2")
-(instances (project "sn64-v2" (path "/d28f46aa-91c7-5060-a563-bf74d208e51e/69e05daa-4082-5d3e-8a2d-0d56f4a78932" (reference "R203") (unit 1)))))
+(instances (project "sn64-v2" (path "/d28f46aa-91c7-5060-a563-bf74d208e51e/69e05daa-4082-5d3e-8a2d-0d56f4a78932" (reference "R204") (unit 1)))))
 (wire (pts (xy 588.01 373.38) (xy 588.01 368.3)) (stroke (width 0) (type default)))
 (global_label "FPGA_3V3" (shape passive) (at 588.01 368.3 90) (fields_autoplaced yes) (effects (font (size 1.016 1.016)) (justify left)) (property "Intersheetrefs" "${INTERSHEET_REFS}" (at 588.01 368.3 0) (effects (font (size 1.27 1.27)) (hide yes))))
 (wire (pts (xy 588.01 381) (xy 588.01 386.08)) (stroke (width 0) (type default)))
-(global_label "CIC_DATA1_OD" (shape passive) (at 588.01 386.08 270) (fields_autoplaced yes) (effects (font (size 1.016 1.016)) (justify right)) (property "Intersheetrefs" "${INTERSHEET_REFS}" (at 588.01 386.08 0) (effects (font (size 1.27 1.27)) (hide yes))))
-(symbol (lib_id "Device:R") (at 603.25 377.19 0) (unit 1) (exclude_from_sim no) (in_bom yes) (on_board yes) (dnp no)
-(property "Reference" "R204" (at 605.79 375.92 0) (effects (font (size 1.27 1.27)) (justify left)))
-(property "Value" "10k" (at 605.79 378.46 0) (effects (font (size 1.27 1.27)) (justify left)))
-(property "Footprint" "Resistor_SMD:R_0603_1608Metric" (at 603.25 377.19 0) (effects (font (size 1.27 1.27)) (hide yes)))
-(property "Datasheet" "" (at 603.25 377.19 0) (effects (font (size 1.27 1.27)) (hide yes)))
-(pin "1")
-(pin "2")
-(instances (project "sn64-v2" (path "/d28f46aa-91c7-5060-a563-bf74d208e51e/69e05daa-4082-5d3e-8a2d-0d56f4a78932" (reference "R204") (unit 1)))))
-(wire (pts (xy 603.25 373.38) (xy 603.25 368.3)) (stroke (width 0) (type default)))
-(global_label "FPGA_3V3" (shape passive) (at 603.25 368.3 90) (fields_autoplaced yes) (effects (font (size 1.016 1.016)) (justify left)) (property "Intersheetrefs" "${INTERSHEET_REFS}" (at 603.25 368.3 0) (effects (font (size 1.27 1.27)) (hide yes))))
-(wire (pts (xy 603.25 381) (xy 603.25 386.08)) (stroke (width 0) (type default)))
-(global_label "RESET_PULL_OD" (shape passive) (at 603.25 386.08 270) (fields_autoplaced yes) (effects (font (size 1.016 1.016)) (justify right)) (property "Intersheetrefs" "${INTERSHEET_REFS}" (at 603.25 386.08 0) (effects (font (size 1.27 1.27)) (hide yes))))
+(global_label "RESET_PULL_OD" (shape passive) (at 588.01 386.08 270) (fields_autoplaced yes) (effects (font (size 1.016 1.016)) (justify right)) (property "Intersheetrefs" "${INTERSHEET_REFS}" (at 588.01 386.08 0) (effects (font (size 1.27 1.27)) (hide yes))))
 (symbol (lib_id "Device:R") (at 27.94 438.15 0) (unit 1) (exclude_from_sim no) (in_bom yes) (on_board yes) (dnp no)
 (property "Reference" "R205" (at 30.48 436.88 0) (effects (font (size 1.27 1.27)) (justify left)))

Commit message: Pre-order review, work in progress: finger fill, U6 footprint, USB-C port from the drawings, parts list numbers, power re-layout started
Checkpoint in the middle of the review, committed at the owner's request. Not a release.

Done and on the board file:
- ground fill taken out of the N64 edge fingers, ground plane extended to the finger vias
  (apply_finger_clearance_v2.py)
- U6 footprint with the exposed pad of its data sheet, R17 moved, leftovers of the first
  routing trimmed, silkscreen labels tidied, part records synced with the schematic
- USB supply capacitance 8.0 uF, selector soft-start 10 nF

Done elsewhere:
- shell: USB-C port from the JAE drawing, the USB-IF plug limits and the SummerCart64 port
- a maker part number on every bought part; yellow-green lamp; 1 uF at each ADC supply pin
- pack_bitstream.py: the FPGA image packed for a fast load, and the whole flash as one file
- make_production_v2.py (its output is not in this commit: it is remade when the board is done)

In progress, schematic ahead of the board:
- the schematic has 12 more small parts (R321, C324, C325, C213-C220, C46) that the makers'
  data sheets ask for; the board file does not have them yet
- apply_power_layout_v2.py and make_power_plan.py lay the power section out again by the
  makers' layout rules; so far only on working copies under build/

Co-Authored-By: Claude Opus 5.5 <noreply@anthropic.com>
Parts:
- added C213, C214, C215, C216, C217, C218, C219, C220: 100nF, Capacitor_SMD:C_0603_1608Metric, symbol Device:C
- C201, C202, C203, C204, C205, C206, C207, C208, C211: LCSC (none) -> C14663; MPN (none) -> CC0603KRX7R9BB104; Manufacturer (none) -> YAGEO
- C209, C210: LCSC (none) -> C45783; MPN (none) -> CL21A226MAQNNNE; Manufacturer (none) -> Samsung Electro-Mechanics
- C212: LCSC (none) -> C15850; MPN (none) -> CL21A106KAYNNNE; Manufacturer (none) -> Samsung Electro-Mechanics
- J1: now left out of the parts list
- R202, R203, R204, R209: LCSC (none) -> C25804; MPN (none) -> 0603WAF1002T5E; Manufacturer (none) -> UNI-ROYAL
- R205, R206, R207, R208: LCSC (none) -> C23162; MPN (none) -> 0603WAF4701T5E; Manufacturer (none) -> UNI-ROYAL
- R210, R211, R212, R213, R214: LCSC (none) -> C25803; MPN (none) -> 0603WAF1003T5E; Manufacturer (none) -> UNI-ROYAL
- U201, U202, U203, U204, U205: Manufacturer (none) -> Texas Instruments
Connections:
- net FPGA_3V3: now also C213.1, C215.1, C217.1, C219.1
- net GND: now also C213.2, C214.2, C215.2, C216.2, C217.2, C218.2, C219.2, C220.2
- net SNES_5V_CART: now also C214.1, C216.1, C218.1, C220.1
Other:
- moved on the sheet: C209, C210
